File: PCB/Amplificador/EtapaSalida.sch (KiCad schematic (older format))
At the start: 49 parts, among them J2 Conector_Alimentacion, J3 Salida, Q16 Q_NMOS_GDS, Q17 Q_NMOS_GDS, U6 UCC20520DWR, U7 LM7812_TO220

Commit message: Generador de onda triangular terminado y ruteado
Parts:
- U6: symbol UCC20520DWR:UCC20520DWR -> Amplificador-rescue:UCC20520DWR-UCC20520DWR
Changed lines of the file:
@@
 	2350 3300 2100 3300
 $Comp
-L UCC20520DWR:UCC20520DWR U6
+L Amplificador-rescue:UCC20520DWR-UCC20520DWR U6
 U 1 1 605A1251
 P 4250 3200
