File: PCB/Amplificador/Realimentador.sch (KiCad schematic (older format))
At the start: 18 parts, among them IC1 AD817, IC2 AD817, J5 Entrada

Commit message: Generador de onda triangular terminado y ruteado
Parts:
- IC1, IC2: symbol AD817:AD817 -> Amplificador-rescue:AD817-AD817
Changed lines of the file:
@@
 $EndDescr
 $Comp
-L AD817:AD817 IC1
+L Amplificador-rescue:AD817-AD817 IC1
 U 1 1 60543779
 P 4400 4850
@@
 $EndComp
 $Comp
-L AD817:AD817 IC2
+L Amplificador-rescue:AD817-AD817 IC2
 U 1 1 60543F5D
 P 4750 1850
