File: PCB/Amplificador/Triangular.sch (KiCad schematic (older format))
At the start: 57 parts, among them J1 Conector_Alimentacion, Q1 BC847, Q10 BC847, Q11 BC857, Q12 BC847, Q13 2N7002, Q14 BC847, Q15 BC857, Q2 BC847, Q3 BC847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

Commit message: Generador de onda triangular terminado y ruteado
Parts:
- U4: symbol SN74LVC2G02DCUR:SN74LVC2G02DCUR -> Amplificador-rescue:SN74LVC2G02DCUR-SN74LVC2G02DCUR
Changed lines of the file:
@@
 	3950 3300 3950 3150
 $Comp
-L SN74LVC2G02DCUR:SN74LVC2G02DCUR U4
+L Amplificador-rescue:SN74LVC2G02DCUR-SN74LVC2G02DCUR U4
 U 1 1 5FA6D9C3
 P 6800 2200
