File: PCB - Rev2/Amplificador_v2/Amplificador_v2.kicad_pcb (KiCad board)
At the start: 2 copper layers, 58 parts, among them J1 Conector alimentacion, Q1 BC847, Q10 BC847, Q11 BC857, Q12 BC847, Q13 2N7002, Q14 BC847, Q15 BC857, Q2 BC847, Q3 BC847, Q4 2N7002, Q5 BC857, Q6 BC847, Q7 BC847, Q8 BC857, Q9 BC857, U1 TL082, U2 LM311, U3 LM311, U4 SN74LVC2G02DCUR

Commit message: Version sin preampli
Parts:
- added C10: 100n, Capacitor_SMD:C_0805_2012Metric, F.Cu at (86.6, 151.6)
- added C11: 100n, Capacitor_SMD:C_0805_2012Metric, F.Cu at (86.6, 148.0)
- added C12: 10u, Capacitor_SMD:CP_Elec_4x5.3, F.Cu at (82.9, 156.0)
- added C13: 10u, Capacitor_SMD:CP_Elec_4x5.3, F.Cu at (82.9, 148.8)
- added C14: 3.3n, Capacitor_SMD:C_0805_2012Metric, F.Cu at (95.9, 156.0)
- added C15: 3.3n, Capacitor_SMD:C_0805_2012Metric, F.Cu at (98.0, 162.2)
- added C16: 1u, Capacitor_THT:C_Radial_D5.0mm_H11.0mm_P2.00mm, F.Cu at (91.9, 160.1)
- added C17: 100n, Capacitor_SMD:C_0805_2012Metric, F.Cu at (98.0, 152.5)
- added C18: 33p, Capacitor_SMD:C_0805_2012Metric, F.Cu at (97.3, 147.3)
- added C19: 100n, Capacitor_SMD:C_0805_2012Metric, B.Cu at (114.0, 151.4)
- added C20: 10u, Capacitor_THT:C_Radial_D4.0mm_H7.0mm_P1.50mm, F.Cu at (119.3, 168.1)
- added C21: 100u, Capacitor_THT:C_Radial_D8.0mm_H11.5mm_P3.50mm, F.Cu at (107.4, 168.0)
- added C22: 1u, Capacitor_SMD:C_0805_2012Metric, B.Cu at (116.3, 151.4)
- added C23: 10u, Capacitor_SMD:C_0805_2012Metric, B.Cu at (116.5, 157.8)
- added C24: 10u, Capacitor_SMD:C_0805_2012Metric, F.Cu at (113.6, 166.9)
- added C25: 220n, Capacitor_SMD:C_0805_2012Metric, B.Cu at (114.2, 157.8)
- added C26: 100n, Capacitor_SMD:C_0805_2012Metric, F.Cu at (113.6, 169.0)
- added C27: 1n, Capacitor_SMD:C_0805_2012Metric, F.Cu at (126.7, 150.6)
- added C28: 1n, Capacitor_SMD:C_0805_2012Metric, F.Cu at (125.5, 164.6)
- added C29: C, Capacitor_SMD:C_1206_3216Metric, F.Cu at (148.9, 149.5)
- added C30: C, Capacitor_SMD:C_1206_3216Metric, F.Cu at (148.9, 163.1)
- added C31: 330n, Capacitor_THT:C_Rect_L18.0mm_W5.0mm_P15.00mm_FKS3_FKP3, F.Cu at (171.0, 163.5)
- added C32: C, Capacitor_SMD:C_1206_3216Metric, F.Cu at (161.5, 168.8)
- added C33: 10u, Capacitor_THT:C_Radial_D4.0mm_H7.0mm_P1.50mm, F.Cu at (101.0, 133.4)
- added C34: 100n, Capacitor_SMD:C_0805_2012Metric, F.Cu at (101.5, 137.9)
- added C35: C, Capacitor_SMD:C_0805_2012Metric, F.Cu at (102.2, 140.5)
- added C36: C, Capacitor_SMD:C_0805_2012Metric, F.Cu at (105.2, 134.1)
- added C37: C, Capacitor_SMD:C_0805_2012Metric, F.Cu at (110.7, 143.6)
- added C38: C, Capacitor_SMD:C_0805_2012Metric, F.Cu at (104.4, 143.6)
- added C39: 3300u, Capacitor_THT:CP_Radial_D18.0mm_P7.50mm, F.Cu at (169.4, 101.7)
- added C40: 3300u, Capacitor_THT:CP_Radial_D18.0mm_P7.50mm, F.Cu at (169.4, 121.8)
- added C41: 3300u, Capacitor_THT:CP_Radial_D18.0mm_P7.50mm, F.Cu at (149.5, 101.7)
- added C42: 3300u, Capacitor_THT:CP_Radial_D18.0mm_P7.50mm, F.Cu at (149.5, 121.7)
- added C43: 100u, Capacitor_THT:CP_Radial_D8.0mm_P3.50mm, F.Cu at (116.2, 115.2)
- added C44: 100u, Capacitor_THT:CP_Radial_D8.0mm_P3.50mm, F.Cu at (135.4, 120.0)
- added C45: 1u, Capacitor_SMD:C_0805_2012Metric, F.Cu at (115.0, 126.3)
- added C46: 1u, Capacitor_SMD:C_0805_2012Metric, F.Cu at (133.9, 114.3)
- added C47: 100u, Capacitor_SMD:CP_Elec_6.3x7.7, F.Cu at (103.8, 124.8)
- added C48: 1u, Capacitor_SMD:C_0805_2012Metric, F.Cu at (128.1, 122.6)
- added C49: 1u, Capacitor_SMD:C_0805_2012Metric, F.Cu at (110.4, 126.3)
- added C50: 100u, Capacitor_SMD:CP_Elec_6.3x7.7, F.Cu at (122.9, 124.3)
- added C51: 100u, Capacitor_SMD:CP_Elec_6.3x7.7, F.Cu at (84.9, 124.5)
- added C52: 1u, Capacitor_SMD:C_0805_2012Metric, F.Cu at (93.0, 118.2)
- added C53: 2200u, Capacitor_THT:CP_Radial_D13.0mm_P5.00mm, F.Cu at (56.2, 91.9)
- added C54: 2200u, Capacitor_THT:CP_Radial_D13.0mm_P5.00mm, F.Cu at (179.1, 155.0)
- added D3: MURS120T3G, Diode_SMD:D_SMB_Handsoldering, B.Cu at (122.4, 152.1)
- added D4: MURS120T3G, Diode_SMD:D_SMB_Handsoldering, F.Cu at (118.7, 151.5)
- added D5: MURS120T3G, Diode_SMD:D_SMB_Handsoldering, F.Cu at (118.7, 157.6)
- added D6: MURS320T3G, Diode_SMD:D_SMC_Handsoldering, F.Cu at (143.8, 145.2)
- added D7: MURS320T3G, Diode_SMD:D_SMC_Handsoldering, F.Cu at (143.8, 160.1)
- added IC1: AD817, Package_SO:SOIC-8_3.9x4.9mm_P1.27mm, F.Cu at (108.0, 138.7)
- added IC2: AD817, Package_SO:SOIC-8_3.9x4.9mm_P1.27mm, F.Cu at (117.8, 138.8)
- added J2: Conector alimentacion, Connector_PinHeader_2.54mm:PinHeader_1x04_P2.54mm_Vertical, F.Cu at (96.6, 134.7)
- added J3: Conn_01x02_Male, Connector_PinHeader_2.54mm:PinHeader_1x02_P2.54mm_Vertical, F.Cu at (70.7, 101.5)
- added J4: Conn_01x03_Male, Connector_PinHeader_2.54mm:PinHeader_1x03_P2.54mm_Vertical, F.Cu at (88.6, 139.3)
- added J5: Conn_01x03_Male, Connector_PinHeader_2.54mm:PinHeader_1x03_P2.54mm_Vertical, F.Cu at (93.7, 143.1)
- added J6: Screw_Terminal_01x02, TerminalBlock:TerminalBlock_bornier-2_P5.08mm, F.Cu at (178.1, 163.0)
- added J7: Conn_01x02_Male, Connector_PinHeader_2.54mm:PinHeader_1x02_P2.54mm_Vertical, F.Cu at (98.7, 143.4)
- added J8: Conn_01x03_Male, Connector_PinHeader_2.54mm:PinHeader_1x03_P2.54mm_Vertical, F.Cu at (123.8, 140.8)
- added J9: Screw_Terminal_01x03, TerminalBlock:TerminalBlock_bornier-3_P5.08mm, F.Cu at (184.5, 110.6)
- added JP2: Jumper, Jumper:SolderJumper-2_P1.3mm_Open_RoundedPad1.0x1.5mm, F.Cu at (91.9, 154.7)
- added JP3: Jumper, Jumper:SolderJumper-2_P1.3mm_Open_RoundedPad1.0x1.5mm, F.Cu at (97.3, 159.1)
- added JP4: Jumper, Jumper:SolderJumper-2_P1.3mm_Open_RoundedPad1.0x1.5mm, F.Cu at (75.2, 101.0)
- added L1: INDUCTOR, footprints:15333C, F.Cu at (155.8, 151.5)
- added Q16: PHB27NQ10T, Package_TO_SOT_SMD:TO-263-2, F.Cu at (133.5, 144.3)
- added Q17: PHB27NQ10T, Package_TO_SOT_SMD:TO-263-2, F.Cu at (133.5, 161.5)
- added R16: 1k, Resistor_SMD:R_0805_2012Metric, F.Cu at (91.9, 157.0)
- added R17: 1k, Resistor_SMD:R_0805_2012Metric, F.Cu at (98.0, 156.0)
- added R18: 1k, Resistor_SMD:R_0805_2012Metric, F.Cu at (95.9, 162.2)
- added R19: 49.9, Resistor_SMD:R_0805_2012Metric, F.Cu at (97.3, 149.5)
- added R20: 10, Resistor_SMD:R_2512_6332Metric, B.Cu at (122.2, 157.5)
- added R21: 1.2, Resistor_SMD:R_0805_2012Metric, F.Cu at (124.6, 150.6)
- added R22: 3.3, Resistor_SMD:R_0805_2012Metric, F.Cu at (125.8, 147.6)
- added R23: 1.2, Resistor_SMD:R_0805_2012Metric, F.Cu at (125.5, 158.6)
- added R24: 3.3, Resistor_SMD:R_0805_2012Metric, F.Cu at (124.8, 161.5)
- added R25: R, Resistor_SMD:R_2512_6332Metric, F.Cu at (149.7, 143.0)
- added R26: R, Resistor_SMD:R_2512_6332Metric, F.Cu at (149.7, 156.7)
- added R27: R, Resistor_SMD:R_2512_6332Metric, F.Cu at (168.8, 168.8)
- added R28: 1k, Resistor_SMD:R_0805_2012Metric, F.Cu at (97.8, 137.9)
- added R29: R, Resistor_SMD:R_0805_2012Metric, F.Cu at (98.6, 140.5)
- added R30: 1k, Resistor_SMD:R_0805_2012Metric, F.Cu at (112.2, 134.9)
- added R31: R, Resistor_SMD:R_0805_2012Metric, F.Cu at (107.2, 134.1)
- added R32: R, Resistor_SMD:R_0805_2012Metric, F.Cu at (108.6, 143.6)
- added R33: 1k, Resistor_SMD:R_0805_2012Metric, F.Cu at (112.9, 139.8)
- added R34: 1k, Resistor_SMD:R_0805_2012Metric, F.Cu at (115.8, 134.9)
- added R35: R, Resistor_SMD:R_0805_2012Metric, F.Cu at (106.5, 143.6)
- added R36: 18k, Resistor_SMD:R_0805_2012Metric, F.Cu at (119.4, 134.9)
- added R37: R, Resistor_SMD:R_2512_6332Metric, F.Cu at (55.4, 101.6)
- added R38: R, Resistor_SMD:R_2512_6332Metric, F.Cu at (64.1, 101.6)
- added TP10: TestPoint, TestPoint:TestPoint_Pad_2.0x2.0mm, F.Cu at (88.5, 156.4)
- added TP11: TestPoint, TestPoint:TestPoint_Pad_2.0x2.0mm, F.Cu at (125.5, 144.8)
- added TP12: TestPoint, TestPoint:TestPoint_Pad_2.0x2.0mm, F.Cu at (125.0, 168.2)
- added U10: LM7805_TO220, Package_TO_SOT_THT:TO-220-3_Vertical, F.Cu at (96.9, 121.3)
- added U5: LM311, Package_SO:SOIC-8_3.9x4.9mm_P1.27mm, F.Cu at (90.6, 149.5)
- added U6: UCC20520DWR, footprints:SOIC127P1030X265-16N, F.Cu at (105.9, 154.4)
- added U7: LM7812_TO220, Package_TO_SOT_THT:TO-220-3_Vertical, F.Cu at (114.6, 164.1)
- added U8: LM7815_TO220, Package_TO_SOT_THT:TO-220-3_Vertical, F.Cu at (116.0, 121.4)
- added U9: LM7915_TO220, Package_TO_SOT_THT:TO-220-3_Vertical, F.Cu at (134.6, 126.4)
- moved C1 111.7 mm to (66.0, 135.7)
- moved C2 111.7 mm to (59.4, 139.3)
- moved C4 111.7 mm to (75.8, 160.7)
- moved C8 111.7 mm to (74.7, 144.4)
- moved D1 111.7 mm to (57.5, 149.0)
- moved D2 111.7 mm to (57.6, 161.5)
- moved Q11 111.7 mm to (51.7, 157.1)
- moved Q12 111.7 mm to (47.8, 157.1)
- moved Q14 111.7 mm to (55.1, 166.5)
- moved Q15 111.7 mm to (47.8, 166.5)
- moved Q3 111.7 mm to (50.1, 143.8)
- moved Q8 111.7 mm to (55.4, 153.4)
- moved Q9 111.7 mm to (55.4, 157.1)
- moved R1 111.7 mm to (58.3, 143.7)
- moved R11 111.7 mm to (51.4, 167.8)
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Routing:
- net GND: track 137.8 -> 603.4 mm, vias 11 -> 34
- net VEE: track 0.00 -> 248.4 mm, vias 0 -> 3
- net VCC: track 4.68 -> 241.6 mm
- net +15V: track 115.5 -> 239.8 mm, vias 2 -> 9
- net +5V: track 35.9 -> 152.6 mm, vias 1 -> 2
- net VS: track 0.00 -> 95.4 mm, vias 0 -> 2
- net -15V: track 0.00 -> 90.4 mm, vias 0 -> 7
- net VOUT: track 0.00 -> 70.5 mm
- net /VDDB: track 0.00 -> 23.3 mm, vias 0 -> 3
- net Net-(C28-Pad1): track 0.00 -> 18.6 mm
- net Net-(C36-Pad1): track 0.00 -> 18.4 mm
- net Error_amplifier_out: track 0.00 -> 16.6 mm
- net /HO: track 0.00 -> 16.1 mm
- net /LO: track 0.00 -> 14.9 mm
- net Net-(C36-Pad2): track 0.00 -> 14.1 mm
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- added copper zone on F.Cu, net +15V
- added copper zone on B.Cu, net +5V
- added copper zone on F.Cu, net +5V
- added copper zone on B.Cu, net -15V
- added copper zone on F.Cu, net -15V
- added copper zone on F.Cu, net /HO
- added copper zone on F.Cu, net /LO
- added copper zone on B.Cu, net /VDDA
- added copper zone on F.Cu, net /VDDA
- added copper zone on B.Cu, net /VDDB
- added copper zone on F.Cu, net /VDDB
- added copper zone on F.Cu, net GND
- added copper zone on F.Cu, net Net-(C14-Pad2)
- added copper zone on F.Cu, net Net-(C18-Pad1)
- added copper zone on F.Cu, net Net-(C27-Pad1)
- added copper zone on F.Cu, net Net-(C28-Pad1)
- added copper zone on F.Cu, net Net-(C29-Pad1)
- added copper zone on F.Cu, net Net-(C30-Pad1)
- added copper zone on B.Cu, net Net-(D3-Pad1)
- added copper zone on F.Cu, net Net-(D4-Pad1)
- added copper zone on F.Cu, net Net-(D5-Pad1)
- added copper zone on F.Cu, net Net-(JP2-Pad1)
- added copper zone on F.Cu, net VCC
- added copper zone on B.Cu, net VEE
- added copper zone on F.Cu, net VEE
- added copper zone on B.Cu, net VS
- added copper zone on F.Cu, net VS
Other:
- board outline added: 150 x 100 mm

Commit message: Finalizada la placa v2
Parts:
- added C55: 10u, Capacitor_SMD:CP_Elec_4x5.3, F.Cu at (50.4, 144.3)
- added C56: 10u, Capacitor_THT:CP_Radial_D5.0mm_P2.00mm, F.Cu at (73.0, 170.4)
- added C57: 10u, Capacitor_THT:CP_Radial_D5.0mm_P2.00mm, F.Cu at (48.7, 157.2)
- added C58: C, Capacitor_SMD:C_0805_2012Metric, F.Cu at (57.1, 104.2)
- added C59: C, Capacitor_SMD:C_0805_2012Metric, F.Cu at (57.8, 114.4)
- added C60: C, Capacitor_SMD:C_0805_2012Metric, F.Cu at (57.1, 91.3)
- added C61: C, Capacitor_SMD:C_0805_2012Metric, F.Cu at (57.1, 94.9)
- added C62: 10u, Capacitor_SMD:CP_Elec_4x5.3, F.Cu at (69.5, 89.6)
- added C63: C, Capacitor_SMD:C_0805_2012Metric, F.Cu at (65.4, 89.3)
- added C64: 10u, Capacitor_THT:CP_Radial_D4.0mm_P1.50mm, F.Cu at (66.6, 84.6)
- added C65: 10u, Capacitor_SMD:CP_Elec_4x5.3, F.Cu at (59.8, 84.7)
- added C66: C, Capacitor_SMD:C_0805_2012Metric, F.Cu at (61.5, 88.4)
- added C67: C, Capacitor_SMD:C_0805_2012Metric, F.Cu at (61.5, 114.4)
- added C68: C, Capacitor_SMD:C_0805_2012Metric, F.Cu at (65.4, 107.3)
- added C69: C, Capacitor_SMD:C_0805_2012Metric, F.Cu at (81.4, 104.6)
- added C70: C, Capacitor_SMD:C_0805_2012Metric, F.Cu at (78.4, 107.5)
- added C71: C, Capacitor_SMD:C_0805_2012Metric, F.Cu at (104.7, 103.0)
- added C72: 10u, Capacitor_SMD:CP_Elec_4x5.3, F.Cu at (62.3, 118.1)
- added C73: 10u, Capacitor_THT:CP_Radial_D4.0mm_P1.50mm, F.Cu at (68.5, 118.1)
- added C74: 10u, Capacitor_SMD:CP_Elec_4x5.3, F.Cu at (69.2, 107.7)
- added J10: Conn_01x02_Male, Connector_PinHeader_2.54mm:PinHeader_1x02_P2.54mm_Vertical, F.Cu at (80.2, 129.9)
- added J11: Screw_Terminal_01x03, TerminalBlock:TerminalBlock_bornier-3_P5.08mm, F.Cu at (51.6, 112.5)
- added J12: Screw_Terminal_01x02, TerminalBlock:TerminalBlock_bornier-2_P5.08mm, F.Cu at (51.6, 95.7)
- added JP5: Jumper_3_Open, Connector_PinHeader_2.54mm:PinHeader_1x03_P2.54mm_Vertical, F.Cu at (73.9, 110.0)
- added JP6: Jumper_Preampli, Jumper:SolderJumper-2_P1.3mm_Open_RoundedPad1.0x1.5mm, F.Cu at (78.2, 112.2)
- added JP7: Jumper, Jumper:SolderJumper-2_P1.3mm_Open_RoundedPad1.0x1.5mm, F.Cu at (185.7, 160.1)
- added R39: R, Resistor_SMD:R_0805_2012Metric, F.Cu at (56.8, 107.8)
- added R40: R, Resistor_SMD:R_0805_2012Metric, F.Cu at (57.1, 111.5)
- added R41: R, Resistor_SMD:R_0805_2012Metric, F.Cu at (57.8, 88.4)
- added R42: R, Resistor_SMD:R_0805_2012Metric, F.Cu at (57.1, 98.4)
- added R43: R, Resistor_SMD:R_0805_2012Metric, F.Cu at (65.4, 97.5)
- added R44: R, Resistor_SMD:R_0805_2012Metric, F.Cu at (60.1, 112.2)
- added R45: R, Resistor_SMD:R_0805_2012Metric, F.Cu at (65.4, 93.2)
- added R46: R, Resistor_SMD:R_0805_2012Metric, F.Cu at (61.4, 98.8)
- added R47: R, Resistor_SMD:R_0805_2012Metric, F.Cu at (63.7, 112.2)
- added R48: R, Resistor_SMD:R_0805_2012Metric, F.Cu at (65.3, 100.4)
- added R49: R, Resistor_SMD:R_0805_2012Metric, F.Cu at (61.4, 101.2)
- added R50: R, Resistor_SMD:R_0805_2012Metric, F.Cu at (57.8, 101.2)
- added R51: R, Resistor_SMD:R_0805_2012Metric, F.Cu at (65.4, 103.6)
- added R52: R, Resistor_SMD:R_0805_2012Metric, F.Cu at (78.5, 105.3)
- added R53: R, Resistor_SMD:R_0805_2012Metric, F.Cu at (78.5, 103.2)
- added R54: R, Resistor_SMD:R_0805_2012Metric, F.Cu at (84.5, 104.6)
- added R55: R, Resistor_SMD:R_0805_2012Metric, F.Cu at (104.7, 105.2)
- added R56: R, Resistor_SMD:R_0805_2012Metric, F.Cu at (82.1, 107.5)
- added REF**: MountingHole_3.2mm_M3, MountingHole:MountingHole_3.2mm_M3, F.Cu at (50.0, 175.5)
- added REF**: MountingHole_3.2mm_M3, MountingHole:MountingHole_3.2mm_M3, F.Cu at (191.0, 175.5)
- added REF**: MountingHole_3.2mm_M3, MountingHole:MountingHole_3.2mm_M3, F.Cu at (191.0, 83.5)
- added REF**: MountingHole_3.2mm_M3, MountingHole:MountingHole_3.2mm_M3, F.Cu at (50.0, 83.5)
- added RV3: R_POT, Potentiometer_THT:Potentiometer_Alps_RK163_Single_Horizontal, F.Cu at (86.7, 94.7)
- added RV4: R_POT, Potentiometer_THT:Potentiometer_Alps_RK163_Single_Horizontal, F.Cu at (124.5, 94.7)
- added RV5: R_POT, Potentiometer_THT:Potentiometer_Alps_RK163_Single_Horizontal, F.Cu at (105.6, 94.7)
- added U11: NE5532, Package_SO:SOIC-8_3.9x4.9mm_P1.27mm, F.Cu at (61.4, 93.7)
- added U12: NE5532, Package_SO:SOIC-8_3.9x4.9mm_P1.27mm, F.Cu at (61.4, 106.2)
- C16: footprint Capacitor_THT:C_Radial_D5.0mm_H11.0mm_P2.00mm -> Capacitor_THT:CP_Radial_D5.0mm_P2.00mm
- C21: footprint Capacitor_THT:C_Radial_D8.0mm_H11.5mm_P3.50mm -> Capacitor_THT:CP_Radial_D8.0mm_P3.50mm
- C3: value 10u -> 100n; footprint Capacitor_SMD:CP_Elec_4x5.3 -> Capacitor_SMD:C_0805_2012Metric
- C6: value 10u -> 220n; footprint Capacitor_SMD:CP_Elec_4x5.3 -> Capacitor_SMD:C_0805_2012Metric
- J1, J2: value Conector alimentacion -> Conn_01x02_Male; footprint Connector_PinHeader_2.54mm:PinHeader_1x04_P2.54mm_Vertical -> Connector_PinHeader_2.54mm:PinHeader_1x02_P2.54mm_Vertical
- Q11, Q12, Q14, Q15, Q5, Q6, Q8, Q9, R11, R12, R14: moved to F.Cu
- TP1, TP2, TP3, TP4, TP5, TP6, TP7, TP8, TP9: footprint TestPoint:TestPoint_Pad_2.0x2.0mm -> TestPoint:TestPoint_Pad_1.0x1.0mm
- moved C53 136.0 mm to (185.6, 133.5), turned to 270 degrees
- moved R37 126.6 mm to (176.5, 138.6), turned to 90 degrees
- moved JP4 124.3 mm to (185.7, 158.0), turned to 180 degrees
- moved R38 123.2 mm to (176.4, 152.2), turned to 270 degrees
- moved J1 46.6 mm to (101.0, 129.7)
- moved J3 36.8 mm to (88.6, 133.7), turned to 90 degrees
- moved C3 31.2 mm to (52.2, 138.7), turned to 90 degrees
- moved C4 30.8 mm to (54.3, 138.7)
- moved Q14 29.0 mm to (77.9, 148.5), turned to 90 degrees
- moved TP8 27.8 mm to (56.6, 137.1), turned to 270 degrees
- moved C43 26.9 mm to (89.5, 111.7), turned to 270 degrees
- moved R11 26.2 mm to (75.9, 158.3), turned to 270 degrees
- moved TP2 25.6 mm to (61.2, 135.8), turned to 270 degrees
- moved Q15 24.8 mm to (68.1, 152.3), turned to 180 degrees
- moved R14 24.8 mm to (71.7, 151.5)
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Connections:
- J1 pad 1: VCC -> +15V
- J1 pad 2: +15V -> GND
- J2 pad 1: GND -> -15V
- J2 pad 2: +15V -> GND
- R15 pad 1: Net-(C8-Pad2) -> Vtriang
Routing:
- net GND: track 603.4 -> 813.2 mm, vias 34 -> 67
- net -15V: track 90.4 -> 184.8 mm, vias 7 -> 13
- net /Vtriang_off: track 92.9 -> 28.1 mm, vias 1 -> 0
- net Net-(C53-Pad2): track 0.00 -> 55.8 mm
- net /Filter_out: track 0.00 -> 50.3 mm
- net Net-(JP6-Pad1): track 0.00 -> 49.8 mm
- net +15V: track 239.8 -> 279.2 mm, vias 9 -> 19
- net Signal_in: track 0.00 -> 31.7 mm
- net Net-(C70-Pad2): track 0.00 -> 26.9 mm
- net VCC: track 241.6 -> 217.1 mm, vias 0 -> 2
- net +5V: track 152.6 -> 129.8 mm
- net Net-(C69-Pad2): track 0.00 -> 21.1 mm
- net /U-: track 32.5 -> 14.2 mm
- net Net-(JP5-Pad1): track 0.00 -> 15.9 mm
- net /U+: track 32.2 -> 18.4 mm, vias 2 -> 0
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- added copper zone on F.Cu, net Net-(C32-Pad1)
- added copper zone on F.Cu, net Net-(C53-Pad2)
- added copper zone on B.Cu, net Net-(Q1-Pad1)
- added copper zone on F.Cu, net Net-(Q1-Pad1)
- added copper zone on F.Cu, net VOUT
Other:
- outline, holes or cut-outs redrawn
- board text added: "-15V"
- board text added: "15V"
- board text added: "5V"
- board text added: "AMPLIFICADOR CLASE D V.2"
- board text added: "GND"
- board text added: "GRUPO 10 CUENCA - 99319 GILCES - 99074 TURTULA - 99544"
- board text added: "OUT"
- board text added: "Sig"
- board text added: "VCC"
- board text added: "VEE"
