File: PCB - Rev2/Amplificador_v2/Amplificador_v2.sch (KiCad schematic (older format))
At the start: 58 parts, among them J1 Conector alimentacion, Q1 BC847, Q10 BC847, Q11 BC857, Q12 BC847, Q13 2N7002, Q14 BC847, Q15 BC857, Q2 BC847, Q3 BC847, Q4 2N7002, Q5 BC857, Q6 BC847, Q7 BC847, Q8 BC857, Q9 BC857, U1 TL082, U2 LM311, U3 LM311, U4 SN74LVC2G02DCUR

Commit message: Version sin preampli
Parts:
- added C10, C11, C17, C19, C26, C34: 100n, Capacitor_SMD:C_0805_2012Metric, symbol Device:C
- added C12, C13: 10u, Capacitor_SMD:CP_Elec_4x5.3, symbol Device:CP
- added C14, C15: 3.3n, Capacitor_SMD:C_0805_2012Metric, symbol Device:C
- added C16: 1u, Capacitor_THT:CP_Radial_D5.0mm_P2.00mm, symbol Device:CP
- added C18: 33p, Capacitor_SMD:C_0805_2012Metric, symbol Device:C
- added C20, C33: 10u, Capacitor_THT:CP_Radial_D4.0mm_P1.50mm, symbol Device:CP
- added C21, C43, C44: 100u, Capacitor_THT:CP_Radial_D8.0mm_P3.50mm, symbol Device:CP
- added C22, C45, C46, C48, C49, C52: 1u, Capacitor_SMD:C_0805_2012Metric, symbol Device:C
- added C23, C24: 10u, Capacitor_SMD:C_0805_2012Metric, symbol Device:C
- added C25: 220n, Capacitor_SMD:C_0805_2012Metric, symbol Device:C
- added C27, C28: 1n, Capacitor_SMD:C_0805_2012Metric, symbol Device:C
- added C29, C30, C32: C, Capacitor_SMD:C_1206_3216Metric, symbol Device:C
- added C31: 330n, Capacitor_THT:C_Rect_L18.0mm_W5.0mm_P15.00mm_FKS3_FKP3, symbol Device:C
- added C35, C36, C37, C38: C, Capacitor_SMD:C_0805_2012Metric, symbol Device:C
- added C39, C40, C41, C42: 3300u, Capacitor_THT:CP_Radial_D18.0mm_P7.50mm, symbol Device:CP
- added C47, C50, C51: 100u, Capacitor_SMD:CP_Elec_6.3x7.7, symbol Device:CP
- added C53, C54: 2200u, Capacitor_THT:CP_Radial_D13.0mm_P5.00mm, symbol Device:CP
- added D3, D4, D5: MURS120T3G, Diode_SMD:D_SMB_Handsoldering, symbol pspice:DIODE
- added D6, D7: MURS320T3G, Diode_SMD:D_SMC_Handsoldering, symbol pspice:DIODE
- added IC1, IC2: AD817, Package_SO:SOIC-8_3.9x4.9mm_P1.27mm, symbol AD817:AD817
- added J2: Conector alimentacion, Connector_PinHeader_2.54mm:PinHeader_1x04_P2.54mm_Vertical, symbol Connector:Conn_01x04_Male
- added J3, J7: Conn_01x02_Male, Connector_PinHeader_2.54mm:PinHeader_1x02_P2.54mm_Vertical, symbol Connector:Conn_01x02_Male
- added J4, J5, J8: Conn_01x03_Male, Connector_PinHeader_2.54mm:PinHeader_1x03_P2.54mm_Vertical, symbol Connector:Conn_01x03_Male
- added J6: Screw_Terminal_01x02, TerminalBlock:TerminalBlock_bornier-2_P5.08mm, symbol Connector:Screw_Terminal_01x02
- added J9: Screw_Terminal_01x03, TerminalBlock:TerminalBlock_bornier-3_P5.08mm, symbol Connector:Screw_Terminal_01x03
- added JP2, JP3, JP4: Jumper, Jumper:SolderJumper-2_P1.3mm_Open_RoundedPad1.0x1.5mm, symbol Jumper:SolderJumper_2_Open
- added L1: INDUCTOR, footprints:15333C, symbol pspice:INDUCTOR
- added Q16, Q17: PHB27NQ10T, Package_TO_SOT_SMD:TO-263-2, symbol Device:Q_NMOS_GDS
- added R16, R17, R18, R28, R30, R33, R34: 1k, Resistor_SMD:R_0805_2012Metric, symbol Device:R
- added R19: 49.9, Resistor_SMD:R_0805_2012Metric, symbol Device:R
- added R20: 10, Resistor_SMD:R_2512_6332Metric, symbol Device:R
- added R21, R23: 1.2, Resistor_SMD:R_0805_2012Metric, symbol Device:R
- added R22, R24: 3.3, Resistor_SMD:R_0805_2012Metric, symbol Device:R
- added R25, R26, R27, R37, R38: R, Resistor_SMD:R_2512_6332Metric, symbol Device:R
- added R29, R31, R32, R35: R, Resistor_SMD:R_0805_2012Metric, symbol Device:R
- added R36: 18k, Resistor_SMD:R_0805_2012Metric, symbol Device:R
- added TP10, TP11, TP12: TestPoint, TestPoint:TestPoint_Pad_2.0x2.0mm, symbol Connector:TestPoint
- added U10: LM7805_TO220, Package_TO_SOT_THT:TO-220-3_Vertical, symbol Regulator_Linear:LM7805_TO220
- added U5: LM311, Package_SO:SOIC-8_3.9x4.9mm_P1.27mm, symbol Comparator:LM311
- added U6: UCC20520DWR, footprints:SOIC127P1030X265-16N, symbol UCC20520DWR:UCC20520DWR
- added U7: LM7812_TO220, Package_TO_SOT_THT:TO-220-3_Vertical, symbol Regulator_Linear:LM7812_TO220
- added U8: LM7815_TO220, Package_TO_SOT_THT:TO-220-3_Vertical, symbol Regulator_Linear:LM7815_TO220
- added U9: LM7915_TO220, Package_TO_SOT_THT:TO-220-3_Vertical, symbol Regulator_Linear:LM7915_TO220
- R15, R5, R7: footprint Resistor_SMD:R_0805_2012Metric -> Resistor_SMD:R_2512_6332Metric
Connections:
- net +15V: now also C10.1, C12.1, C33.1, C34.1, C47.1, C49.1, IC1.7, IC2.7, J2.2 (Pin_2), U10.1 (VI), U5.8 (V+), U8.3 (VO)
- net +5V: now also C14.1, C16.1, C17.1, C51.1, C52.1, J2.4 (Pin_4), R16.1, U10.3 (VO), U6.3 (VCCI-1), U6.8 (VCCI)
- net GND: now also C10.2, C11.1, C12.2, C13.1, C15.2, C16.2, C17.2, C18.2, C21.1, C24.1, C26.1, C31.2, C32.2, C35.1, C37.2, C39.2, C40.1, C41.2, C42.1, C43.2, C44.1, C45.2, C46.1, C47.2, C48.1, C49.2, C50.1, C51.2, C52.2, C54.2, J2.1 (Pin_1), J3.2 (Pin_2), J9.2 (Pin_2), JP3.1 (A), JP4.1 (A), R17.2, R18.2, R29.2, R33.2, R38.1, U10.2 (GND), U5.1 (GND), U6.4 (GND), U7.1 (VI), U8.2 (GND), U9.1 (GND)
- net VCC: now also C39.1, C41.1, C43.1, C45.1, C53.1, D6.2 (A), J9.1 (Pin_1), Q16.2 (D), R25.2, R37.2, U8.1 (VI)
- net Vtriang: now also U5.3 (-)
- new net: J5.2 (Pin_2), U5.2 (+)
- new net: JP2.1 (A), R16.2, TP10.1, U5.7
- new net: J4.1 (Pin_1), J5.3 (Pin_3)
- new net: C18.1, R19.2, U6.1 (PWM)
- new net: C14.2, JP3.2 (B), R17.1, U6.5 (DISABLE)
- new net: C15.1, R18.1, U6.6 (DT)
- new net: C53.2, C54.1, J6.2 (Pin_2), JP4.2 (B), R37.1, R38.2
- new net: D3.1 (K), R20.1
- new net: D4.1 (K), R21.1
- new net: C27.1, Q16.1 (G), R21.2, R22.2, TP11.1
- new net: D5.1 (K), R23.1
- new net: C28.1, Q17.1 (G), R23.2, R24.2, TP12.1
- new net: C29.1, R25.1
- new net: C30.1, R26.1
- new net: C32.1, R27.1
- new net: IC2.2, IC2.6, R30.1
- new net: IC2.3, R33.1, R34.2
- new net: R34.1, R36.2
- new net: J8.2 (Pin_2), R36.1
- new net: C36.2, IC1.2, R30.2, R31.1
- new net: C36.1, C38.2, IC1.6, J7.2 (Pin_2), R31.2, R35.1
- new net: C35.2, IC1.3, R28.2, R29.1
- new net: C37.1, R32.1
- new net -15V: C11.2, C13.2, C33.2, C34.2, C48.2, C50.2, IC1.4, IC2.4, J2.3 (Pin_3), U5.4 (V-), U9.3 (VO)
- new net Error_amplifier_in: J4.3 (Pin_3), R28.1
- new net Error_amplifier_out: C38.1, J5.1 (Pin_1), J7.1 (Pin_1), R32.2, R35.2
- new net HO: D4.2 (A), R22.1, U6.15 (OUTA)
- new net LO: D5.2 (A), R24.1, U6.10 (OUTB)
- new net PWM: JP2.2 (B), R19.1
- new net Signal_in: J3.1 (Pin_1), J4.2 (Pin_2)
- new net VDDA: C19.1, C22.1, D3.2 (A), U6.16 (VDDA)
- new net VDDB: C20.1, C23.1, C25.1, R20.2, U6.11 (VDDB), U7.3 (VO)
- new net VEE: C20.2, C21.2, C23.2, C24.2, C25.2, C26.2, C28.2, C30.2, C40.2, C42.2, C44.2, C46.2, D7.1 (K), J9.3 (Pin_3), Q17.3 (S), U6.9 (VSSB), U7.2 (GND), U9.2 (VI)
- new net VOUT: C31.1, J6.1 (Pin_1), J8.3 (Pin_3), L1.2, R27.2
- new net VS: C19.2, C22.2, C27.2, C29.2, D6.1 (K), D7.2 (A), J8.1 (Pin_1), L1.1, Q16.3 (S), Q17.2 (D), R26.2, U6.14 (VSSA)
Other:
- note added: "ALIMENTACION"
- note added: "BOOTSTRAP"
- note added: "Bypass \n(cerca de \nentrada)"
- note added: "Bypass \n(cerca de reguladores)"
- note added: "Dead Time"
- note added: "ETAPA DE SALIDA"
- note added: "Filtro PWM"
- note added: "GENERADOR DE PWM\n"
- note added: "REALIMENTADOR"
- note added: "Red de adelanto-atraso opcional"
- note added: "Snubber"
- note added: "Startup protection"
- moved on the sheet: C1, C2, C3, C4, C5, C6, C7, C8, C9, D1, D2, J1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

Commit message: Finalizada la placa v2
Parts:
- removed C3, C6: 10u, Capacitor_SMD:CP_Elec_4x5.3, symbol Device:CP
- removed J1, J2: Conector alimentacion, Connector_PinHeader_2.54mm:PinHeader_1x04_P2.54mm_Vertical, symbol Connector:Conn_01x04_Male
- added C3: 100n, Capacitor_SMD:C_0805_2012Metric, symbol Device:C
- added C55, C62, C65, C72, C74: 10u, Capacitor_SMD:CP_Elec_4x5.3, symbol Device:CP
- added C56, C57: 10u, Capacitor_THT:CP_Radial_D5.0mm_P2.00mm, symbol Device:CP
- added C58, C59, C60, C61, C63, C66, C67, C68, C69, C70, C71: C, Capacitor_SMD:C_0805_2012Metric, symbol Device:C
- added C6: 220n, Capacitor_SMD:C_0805_2012Metric, symbol Device:C
- added C64, C73: 10u, Capacitor_THT:CP_Radial_D4.0mm_P1.50mm, symbol Device:CP
- added J1, J10, J2: Conn_01x02_Male, Connector_PinHeader_2.54mm:PinHeader_1x02_P2.54mm_Vertical, symbol Connector:Conn_01x02_Male
- added J11: Screw_Terminal_01x03, TerminalBlock:TerminalBlock_bornier-3_P5.08mm, symbol Connector:Screw_Terminal_01x03
- added J12: Screw_Terminal_01x02, TerminalBlock:TerminalBlock_bornier-2_P5.08mm, symbol Connector:Screw_Terminal_01x02
- added JP5: Jumper_3_Open, Connector_PinHeader_2.54mm:PinHeader_1x03_P2.54mm_Vertical, symbol Jumper:Jumper_3_Open
- added JP6: Jumper_Preampli, Jumper:SolderJumper-2_P1.3mm_Open_RoundedPad1.0x1.5mm, symbol Jumper:SolderJumper_2_Open
- added JP?: Jumper, Jumper:SolderJumper-2_P1.3mm_Open_RoundedPad1.0x1.5mm, symbol Jumper:SolderJumper_2_Open
- added R39, R40, R41, R42, R43, R44, R45, R46, R47, R48, R49, R50, R51, R52, R53, R54, R55, R56: R, Resistor_SMD:R_0805_2012Metric, symbol Device:R
- added RV3, RV4, RV5: R_POT, Potentiometer_THT:Potentiometer_Alps_RK163_Single_Horizontal, symbol Device:R_POT
- added U11, U12: NE5532, Package_SO:SOIC-8_3.9x4.9mm_P1.27mm, symbol Amplifier_Operational:NE5532
- R15, R5, R7: footprint Resistor_SMD:R_2512_6332Metric -> Resistor_SMD:R_0805_2012Metric
- TP1, TP2, TP3, TP4, TP5, TP6, TP7, TP8, TP9: footprint TestPoint:TestPoint_Pad_2.0x2.0mm -> TestPoint:TestPoint_Pad_1.0x1.0mm
Connections:
- net +15V: now also C3.1, C62.1, C63.1, C64.1, C67.1, C72.1, C73.1, J1.1 (Pin_1), U11.8 (V+), U12.8 (V+)
- net +5V: now also C55.1, C56.1, C57.1, C6.1, J10.1 (Pin_1)
- net -15V: now also C64.2, C65.2, C66.1, C68.1, C73.2, C74.2, J2.1 (Pin_1), U11.4 (V-), U12.4 (V-)
- net GND: now also C3.2, C55.2, C56.2, C57.2, C6.2, C62.2, C63.2, C65.1, C66.2, C67.2, C68.2, C71.2, C72.2, C74.1, J1.2 (Pin_2), J10.2 (Pin_2), J11.2 (Pin_2), J2.2 (Pin_2), JP?.1 (A), R41.2, R42.2, R50.1, R53.2, R55.2, U12.5 (+)
- net Signal_in: now also JP6.2 (B)
- net Vtriang: now also R15.1
- net at C8.2, C9.2, JP1.1 (A)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: no longer R15.1
- net at C53.2, C54.1, J6.2 (Pin_2)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: now also JP?.2 (B)
- new net: C60.1, R41.1, U11.3 (+)
- new net: R45.2, R48.1, U11.1
- new net: R43.1, R45.1, U11.2 (-)
- new net: C61.1, R42.1, U11.5 (+)
- new net: R43.2, R46.1, U11.6 (-)
- new net: R46.2, R49.1, U11.7
- new net: R49.2, R50.2, U12.3 (+)
- new net: R48.2, R51.1, U12.2 (-)
- new net: JP5.3 (B), R51.2, U12.1
- new net: C58.1, R39.1
- new net: R39.2, R40.2, R44.1
- new net: C59.1, R40.1
- new net: R44.2, R47.1, U12.6 (-)
- new net: JP5.1 (A), R47.2, U12.7
- new net: C69.2, R52.2, R54.1, RV3.1, RV3.2
- new net: C69.1, R53.1, RV3.3
- new net: C70.2, R56.2, RV5.2, RV5.3
- new net: C71.1, RV5.1
- new net: JP6.1 (A), R55.1, RV4.2, RV4.3
- new net Filter_in: C70.1, JP5.2 (C), R52.1
- new net Filter_out: R54.2, R56.1, RV4.1
- new net In+: C60.2, J12.2 (Pin_2)
- new net In-: C61.2, J12.1 (Pin_1)
- new net Left: C59.2, J11.1 (Pin_1)
- new net Right: C58.2, J11.3 (Pin_3)
Other:
- moved on the sheet: J5, R15

Commit message: Placa finalizada y lista para enviar
Parts:
- added RV6: 10k, Potentiometer_THT:Potentiometer_Bourns_3296W_Vertical, symbol Device:R_POT_TRIM
- R3: value 12k -> 5.6k
- RV3, RV4, RV5: footprint Potentiometer_THT:Potentiometer_Alps_RK163_Single_Horizontal -> footprints:Potentiometer_Alps_RK163_Single_Horizontal
- gave numbers to parts that had none: 1
Connections:
- net VCC: now also RV6.1; no longer R3.2
- net In+ renamed IN+
- net In- renamed IN-
- net Left renamed LEFT
- net Right renamed RIGHT
- new net: R3.2, RV6.2, RV6.3
- no-connect marks 0 -> 10
Other:
- note removed: "ALIMENTACION"
- moved on the sheet: J11, R1, R2
Changed lines of the file:
@@
 L Device:R R1
 U 1 1 60D49C24
-P 4000 21100
-F 0 "R1" H 4070 21146 50  0000 L CNN
-F 1 "100k" H 4070 21055 50  0000 L CNN
-F 2 "Resistor_SMD:R_0805_2012Metric" V 3930 21100 50  0001 C CNN
-F 3 "~" H 4000 21100 50  0001 C CNN
-	1    4000 21100
+P 4350 21150
+F 0 "R1" H 4420 21196 50  0000 L CNN
+F 1 "100k" H 4420 21105 50  0000 L CNN
+F 2 "Resistor_SMD:R_0805_2012Metric" V 4280 21150 50  0001 C CNN
+F 3 "~" H 4350 21150 50  0001 C CNN
+	1    4350 21150
 	1    0    0    -1
 $EndComp
@@
 L Device:R R2
 U 1 1 60D64FA2
-P 4000 21550
-F 0 "R2" H 4070 21596 50  0000 L CNN
-F 1 "100k" H 4070 21505 50  0000 L CNN
-F 2 "Resistor_SMD:R_0805_2012Metric" V 3930 21550 50  0001 C CNN
-F 3 "~" H 4000 21550 50  0001 C CNN
-	1    4000 21550
+P 4350 21600
+F 0 "R2" H 4420 21646 50  0000 L CNN
+F 1 "100k" H 4420 21555 50  0000 L CNN
+F 2 "Resistor_SMD:R_0805_2012Metric" V 4280 21600 50  0001 C CNN
+F 3 "~" H 4350 21600 50  0001 C CNN
+	1    4350 21600
 	1    0    0    -1
 $EndComp
@@
 P 4000 22700
 F 0 "R3" H 4070 22746 50  0000 L CNN
-F 1 "12k" H 4070 22655 50  0000 L CNN
+F 1 "5.6k" H 4070 22655 50  0000 L CNN
 F 2 "Resistor_SMD:R_0805_2012Metric" V 3930 22700 50  0001 C CNN
 F 3 "~" H 4000 22700 50  0001 C CNN
@@
 $EndComp
 Wire Wire Line
-	4000 21350 4000 21250
-Wire Wire Line
-	4000 21400 4000 21350
-Connection ~ 4000 21350
-Wire Wire Line
 	5000 21850 5000 22000
 Wire Wire Line
@@
 L power:+15V #PWR01
 U 1 1 60E2FEFD
-P 4000 20850
-F 0 "#PWR01" H 4000 20700 50  0001 C CNN
-F 1 "+15V" H 4015 21023 50  0000 C CNN
-F 2 "" H 4000 20850 50  0001 C CNN
-F 3 "" H 4000 20850 50  0001 C CNN
-	1    4000 20850
+P 4350 20900
+F 0 "#PWR01" H 4350 20750 50  0001 C CNN
+F 1 "+15V" H 4365 21073 50  0000 C CNN
+F 2 "" H 4350 20900 50  0001 C CNN
+F 3 "" H 4350 20900 50  0001 C CNN
+	1    4350 20900
 	1    0    0    -1
 $EndComp
@@
 L power:VCC #PWR03
 U 1 1 60E33B18
-P 4000 22400
-F 0 "#PWR03" H 4000 22250 50  0001 C CNN
-F 1 "VCC" H 4017 22573 50  0000 C CNN
-F 2 "" H 4000 22400 50  0001 C CNN
-F 3 "" H 4000 22400 50  0001 C CNN
-	1    4000 22400
+P 4000 21800
+F 0 "#PWR03" H 4000 21650 50  0001 C CNN
+F 1 "VCC" H 4017 21973 50  0000 C CNN
+F 2 "" H 4000 21800 50  0001 C CNN
+F 3 "" H 4000 21800 50  0001 C CNN
+	1    4000 21800
 	1    0    0    -1
 $EndComp
@@
 L power:GND #PWR02
 U 1 1 60E353C5
-P 4000 21800
-F 0 "#PWR02" H 4000 21550 50  0001 C CNN
-F 1 "GND" H 4005 21627 50  0000 C CNN
-F 2 "" H 4000 21800 50  0001 C CNN
-F 3 "" H 4000 21800 50  0001 C CNN
-	1    4000 21800
+P 4350 21850
+F 0 "#PWR02" H 4350 21600 50  0001 C CNN
+F 1 "GND" H 4355 21677 50  0000 C CNN
+F 2 "" H 4350 21850 50  0001 C CNN
+F 3 "" H 4350 21850 50  0001 C CNN
+	1    4350 21850
 	1    0    0    -1
 $EndComp
@@
 	4500 22650 4500 22800
 Wire Wire Line
-	4000 22400 4000 22550
-Wire Wire Line
 	5150 20800 5150 20850
 Wire Wire Line
-	4000 21700 4000 21800
+	4350 21750 4350 21850
 Wire Wire Line
-	4000 20850 4000 20950
+	4350 20900 4350 21000
 $Comp
 L power:GND #PWR016
@@
 $EndComp
 Wire Wire Line
-	4000 21350 5100 21350
-Wire Wire Line
 	5000 21850 4650 21850
 Wire Wire Line
@@
 Text Notes 8100 14500 0    50   ~ 0
 Bypass \n(cerca de \nentrada)
-Text Notes 6200 13550 0    394  ~ 0
-ALIMENTACION
 Wire Notes Line
 	5350 12600 15450 12600
@@
 	6800 15450 6800 16050
 Wire Wire Line
-	6800 16050 7950 16050
+	6800 16050 7250 16050
 Connection ~ 7950 16050
 Wire Wire Line
-	7800 15350 6800 15350
+	7800 15350 7250 15350
 Connection ~ 7800 15350
 Wire Wire Line
 	6800 15250 6800 14650
 Wire Wire Line
-	6800 14650 7950 14650
+	6800 14650 7250 14650
 Connection ~ 7950 14650
 Wire Wire Line
@@
 F 0 "RV3" H 11281 8896 50  0000 R CNN
 F 1 "R_POT" H 11281 8805 50  0000 R CNN
-F 2 "Potentiometer_THT:Potentiometer_Alps_RK163_Single_Horizontal" H 11350 8850 50  0001 C CNN
+F 2 "footprints:Potentiometer_Alps_RK163_Single_Horizontal" H 11350 8850 50  0001 C CNN
 F 3 "~" H 11350 8850 50  0001 C CNN
 	1    11350 8850
@@
 F 0 "RV5" H 13481 8896 50  0000 R CNN
 F 1 "R_POT" H 13481 8805 50  0000 R CNN
-F 2 "Potentiometer_THT:Potentiometer_Alps_RK163_Single_Horizontal" H 13550 8850 50  0001 C CNN
+F 2 "footprints:Potentiometer_Alps_RK163_Single_Horizontal" H 13550 8850 50  0001 C CNN
 F 3 "~" H 13550 8850 50  0001 C CNN
 	1    13550 8850
@@
 F 0 "RV4" H 12431 9546 50  0000 R CNN
 F 1 "R_POT" H 12431 9455 50  0000 R CNN
-F 2 "Potentiometer_THT:Potentiometer_Alps_RK163_Single_Horizontal" H 12500 9500 50  0001 C CNN
+F 2 "footprints:Potentiometer_Alps_RK163_Single_Horizontal" H 12500 9500 50  0001 C CNN
 F 3 "~" H 12500 9500 50  0001 C CNN
 	1    12500 9500
@@
 Text Label 11150 7350 0    50   ~ 0
 Filter_in
-Text GLabel 5750 7050 0    50   Input ~ 0
-In-
-Wire Wire Line
-	5750 7050 6000 7050
-Text GLabel 5750 5250 0    50   Input ~ 0
-In+
-Wire Wire Line
-	5750 5250 6000 5250
-Text GLabel 6250 9200 0    50   Input ~ 0
-Left
-Text GLabel 6250 8550 0    50   Input ~ 0
-Right
-Wire Wire Line
-	6250 8550 6350 8550
-Wire Wire Line
-	6250 9200 6350 9200
 Wire Wire Line
 	5350 6000 6000 6000
 Wire Wire Line
 	6000 6000 6000 5250
-Connection ~ 6000 5250
 Wire Wire Line
 	5350 6100 6000 6100
 Wire Wire Line
 	6000 6100 6000 7050
-Connection ~ 6000 7050
-Connection ~ 6350 8550
-Wire Wire Line
-	6350 8550 6400 8550
-Wire Wire Line
-	6350 8950 6350 9200
-Connection ~ 6350 9200
-Wire Wire Line
-	6350 9200 6400 9200
 Wire Wire Line
 	11350 8200 11350 8650
-Wire Wire Line
-	6350 8250 6350 8550
 $Comp
 L power:GND #PWR06
 U 1 1 5FC9EB8E
-P 5600 8700
-F 0 "#PWR06" H 5600 8450 50  0001 C CNN
-F 1 "GND" H 5605 8527 50  0000 C CNN
-F 2 "" H 5600 8700 50  0001 C CNN
-F 3 "" H 5600 8700 50  0001 C CNN
-	1    5600 8700
+P 5600 8950
+F 0 "#PWR06" H 5600 8700 50  0001 C CNN
+F 1 "GND" H 5605 8777 50  0000 C CNN
+F 2 "" H 5600 8950 50  0001 C CNN
+F 3 "" H 5600 8950 50  0001 C CNN
+	1    5600 8950
 	1    0    0    -1
 $EndComp
 Wire Wire Line
-	5600 8700 5600 8600
+	5600 8950 5600 8850
 $Comp
 L Jumper:SolderJumper_2_Open JP6
@@
 L Connector:Screw_Terminal_01x03 J11
 U 1 1 62C53ECF
-P 5100 8600
-F 0 "J11" H 5018 8917 50  0000 C CNN
-F 1 "Screw_Terminal_01x03" H 5018 8826 50  0000 C CNN
-F 2 "TerminalBlock:TerminalBlock_bornier-3_P5.08mm" H 5100 8600 50  0001 C CNN
-F 3 "~" H 5100 8600 50  0001 C CNN
-	1    5100 8600
+P 5100 8850
+F 0 "J11" H 5018 9167 50  0000 C CNN
+F 1 "Screw_Terminal_01x03" H 5018 9076 50  0000 C CNN
+F 2 "TerminalBlock:TerminalBlock_bornier-3_P5.08mm" H 5100 8850 50  0001 C CNN
+F 3 "~" H 5100 8850 50  0001 C CNN
+	1    5100 8850
 	-1   0    0    1
 $EndComp
 Wire Wire Line
-	5600 8600 5300 8600
-Wire Wire Line
-	5350 8950 5350 8700
-Wire Wire Line
-	5350 8700 5300 8700
-Wire Wire Line
-	5350 8950 6350 8950
-Wire Wire Line
-	5300 8500 5350 8500
-Wire Wire Line
-	5350 8500 5350 8250
-Wire Wire Line
-	5350 8250 6350 8250
+	5600 8850 5300 8850
 Wire Wire Line
 	11350 10450 11350 11150
@@
 	10850 3950 10850 4250
 $Comp
-L Jumper:SolderJumper_2_Open JP?
+L Jumper:SolderJumper_2_Open JP7
 U 1 1 656946C7
 P 41750 24200
-F 0 "JP?" H 41750 24405 50  0000 C CNN
+F 0 "JP7" H 41750 24405 50  0000 C CNN
 F 1 "Jumper" H 41750 24314 50  0000 C CNN
 F 2 "Jumper:SolderJumper-2_P1.3mm_Open_RoundedPad1.0x1.5mm" H 41750 24200 50  0001 C CNN
@@
 Wire Wire Line
 	41750 24550 42150 24550
+$Comp
+L power:PWR_FLAG #FLG0102
+U 1 1 66100454
+P 7250 16050
+F 0 "#FLG0102" H 7250 16125 50  0001 C CNN
+F 1 "PWR_FLAG" H 7250 16223 50  0000 C CNN
+F 2 "" H 7250 16050 50  0001 C CNN
+F 3 "~" H 7250 16050 50  0001 C CNN
+	1    7250 16050
+	-1   0    0    1
+$EndComp
+NoConn ~ 21900 16400
+NoConn ~ 21900 17000
+NoConn ~ 22000 14450
+NoConn ~ 22000 15050
+Text Label 6200 5250 0    50   ~ 0
+IN+
+Text Label 6250 7050 0    50   ~ 0
+IN-
+Text Label 5750 8550 0    50   ~ 0
+RIGHT
+Text Label 5900 9200 0    50   ~ 0
+LEFT
+Wire Wire Line
+	5350 9200 6400 9200
+Wire Wire Line
+	5350 8550 6400 8550
+Wire Wire Line
+	5300 8750 5350 8750
+Wire Wire Line
+	5350 8750 5350 8550
+Wire Wire Line
+	5300 8950 5350 8950
+Wire Wire Line
+	5350 8950 5350 9200
+NoConn ~ 6850 23000
+NoConn ~ 6950 23000
+NoConn ~ 6850 21850
+NoConn ~ 6950 21850
+NoConn ~ 23150 22300
+NoConn ~ 23050 22300
+$Comp
+L power:PWR_FLAG #FLG0104
+U 1 1 66518285
+P 7250 14650
+F 0 "#FLG0104" H 7250 14725 50  0001 C CNN
+F 1 "PWR_FLAG" H 7250 14823 50  0000 C CNN
+F 2 "" H 7250 14650 50  0001 C CNN
+F 3 "~" H 7250 14650 50  0001 C CNN
+	1    7250 14650
+	-1   0    0    1
+$EndComp
+$Comp
+L power:PWR_FLAG #FLG0101
+U 1 1 680E05D9
+P 7250 15350
+F 0 "#FLG0101" H 7250 15425 50  0001 C CNN
+F 1 "PWR_FLAG" H 7250 15523 50  0000 C CNN
+F 2 "" H 7250 15350 50  0001 C CNN
+F 3 "~" H 7250 15350 50  0001 C CNN
+	1    7250 15350
+	-1   0    0    1
+$EndComp
+Connection ~ 7250 15350
+Wire Wire Line
+	7250 15350 6800 15350
+Connection ~ 7250 14650
+Wire Wire Line
+	7250 14650 7950 14650
+Connection ~ 7250 16050
+Wire Wire Line
+	7250 16050 7950 16050
+$Comp
+L Device:R_POT_TRIM RV6
+U 1 1 683BA68F
+P 4000 22250
+F 0 "RV6" H 3930 22296 50  0000 R CNN
+F 1 "10k" H 3930 22205 50  0000 R CNN
+F 2 "Potentiometer_THT:Potentiometer_Bourns_3296W_Vertical" H 4000 22250 50  0001 C CNN
+F 3 "~" H 4000 22250 50  0001 C CNN
+	1    4000 22250
+	1    0    0    -1
+$EndComp
+Wire Wire Line
+	4350 21300 4350 21350
+Wire Wire Line
+	4350 21350 5100 21350
+Connection ~ 4350 21350
+Wire Wire Line
+	4350 21350 4350 21450
+Wire Wire Line
+	4150 22250 4250 22250
+Wire Wire Line
+	4250 22250 4250 22450
+Wire Wire Line
+	4250 22450 4000 22450
+Wire Wire Line
+	4000 22450 4000 22400
+Wire Wire Line
+	4000 22450 4000 22550
+Connection ~ 4000 22450
+Wire Wire Line
+	4000 22100 4000 21800
 $EndSCHEMATC

Commit message: Terminado esto
Parts:
- R18: value 1k -> 2.7k
Changed lines of the file:
@@
 	18250 18950 18250 25450
 Wire Notes Line
-	18250 25450 3600 25450
-Wire Notes Line
 	3600 25450 3600 18950
 Text Notes 7600 19600 0    394  ~ 0
@@
 P 28500 23000
 F 0 "R18" H 28570 23046 50  0000 L CNN
-F 1 "1k" H 28570 22955 50  0000 L CNN
+F 1 "2.7k" H 28570 22955 50  0000 L CNN
 F 2 "Resistor_SMD:R_0805_2012Metric" V 28430 23000 50  0001 C CNN
 F 3 "~" H 28500 23000 50  0001 C CNN
@@
 Wire Wire Line
 	4000 22100 4000 21800
+Wire Notes Line
+	18250 25450 3600 25450
 $EndSCHEMATC

Commit message: Aprobamos
Parts:
- removed C32: C, Capacitor_SMD:C_1206_3216Metric, symbol Device:C
- removed C53, C54: 2200u, Capacitor_THT:CP_Radial_D13.0mm_P5.00mm, symbol Device:CP
- removed JP4, JP7: Jumper, Jumper:SolderJumper-2_P1.3mm_Open_RoundedPad1.0x1.5mm, symbol Jumper:SolderJumper_2_Open
- removed R27, R37, R38: R, Resistor_SMD:R_2512_6332Metric, symbol Device:R
- added C?: 2.2n, Capacitor_SMD:C_0805_2012Metric, symbol Device:C
- C14: value 3.3n -> 10U
- C35, C36: value C -> 2.2n
- C58, C59, C60, C61: value C -> 10u
- C63, C66, C67, C68: value C -> 100n
- R15: value R -> 1K
- R17: value 1k -> 10K
- R18: value 2.7k -> 5.6K
- R20: value 10 -> 0
- R22, R24: value 3.3 -> 4.7
- R29, R31: value R -> 100K
- R39: value R -> 33k
- R40, R44, R48, R49: value R -> 18k
- R41, R42: value R -> 47k
- R43, R50, R51: value R -> 2.7k
- R45, R46: value R -> 1k
- R47: value R -> 25.5k
Connections:
- net GND: now also J6.2 (Pin_2), C?.2
- net at IC2.3, R33.1, R34.2: now also C?.1
Other:
- moved on the sheet: C29, C30, C31, D6, D7, J6, J8, L1, Q16, Q17, R25, R26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
